Commit message: chenged model

File: model/t960a.urdf.xacro (robot description, xacro)
@@ -9,5 +9,5 @@
     <parent link="base_link"/>
     <child link="mobile_wx250s/base_link"/>
-    <origin xyz="0.4265 0 -0.063" rpy="3.14 0 0"/>
+    <origin xyz="0.4265 0 -0.0845" rpy="3.14 0 0"/>
   </joint>
 </robot>
