Commit message: Real hardware integration is ready

File: model/wx250s.urdf (robot description, URDF)
Before this commit: robot mobile_wx250s, 14 links, 13 joints
Links:
- link mobile_wx250s/base_link: geometry collision mesh filename=package://clik1_node_pkg/model/meshes/mobile_wx250s_meshes/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 scale=0.001 0.001 0.001; visual mesh filename=package://clik1_node_pkg/model/meshes/mobile_wx250s_meshes/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 scale=0.001 0.001 0.001
- link mobile_wx250s/gripper_bar_link: geometry collision mesh filename=package://clik1_node_pkg/model/meshes/mobile_wx250s_meshes/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 scale=0.001 0.001 0.001; visual mesh filename=package://clik1_node_pkg/model/meshes/mobile_wx250s_meshes/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 scale=0.001 0.001 0.001
- link mobile_wx250s/gripper_link: geometry collision mesh filename=package://clik1_node_pkg/model/meshes/mobile_wx250s_meshes/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 scale=0.001 0.001 0.001; visual mesh filename=package://clik1_node_pkg/model/meshes/mobile_wx250s_meshes/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 scale=0.001 0.001 0.001
- link mobile_wx250s/gripper_prop_link: geometry collision mesh filename=package://clik1_node_pkg/model/meshes/mobile_wx250s_meshes/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 scale=0.001 0.001 0.001; visual mesh filename=package://clik1_node_pkg/model/meshes/mobile_wx250s_meshes/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 scale=0.001 0.001 0.001
- link mobile_wx250s/left_finger_link: geometry collision mesh filename=package://clik1_node_pkg/model/meshes/mobile_wx250s_meshes/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 scale=0.001 0.001 0.001; visual mesh filename=package://clik1_node_pkg/model/meshes/mobile_wx250s_meshes/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 scale=0.001 0.001 0.001
- link mobile_wx250s/lower_forearm_link: geometry collision mesh filename=package://clik1_node_pkg/model/meshes/mobile_wx250s_meshes/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 scale=0.001 0.001 0.001; visual mesh filename=package://clik1_node_pkg/model/meshes/mobile_wx250s_meshes/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 scale=0.001 0.001 0.001
- link mobile_wx250s/right_finger_link: geometry collision mesh filename=package://clik1_node_pkg/model/meshes/mobile_wx250s_meshes/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 scale=0.001 0.001 0.001; visual mesh filename=package://clik1_node_pkg/model/meshes/mobile_wx250s_10_grip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 scale=0.001 0.001 0.001
- link mobile_wx250s/shoulder_link: geometry collision mesh filename=package://clik1_node_pkg/model/meshes/mobile_wx250s_meshes/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 scale=0.001 0.001 0.001; visual mesh filename=package://clik1_node_pkg/model/meshes/mobile_wx250s_meshes/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 scale=0.001 0.001 0.001
- link mobile_wx250s/upper_arm_link: geometry collision mesh filename=package://clik1_node_pkg/model/meshes/mobile_wx250s_meshes/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 scale=0.001 0.001 0.001; visual mesh filename=package://clik1_node_pkg/model/meshes/mobile_wx250s_meshes/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 scale=0.001 0.001 0.001
- link mobile_wx250s/upper_forearm_link: geometry collision mesh filename=package://clik1_node_pkg/model/meshes/mobile_wx250s_meshes/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 scale=0.001 0.001 0.001; visual mesh filename=package://clik1_node_pkg/model/meshes/mobile_wx250s_meshes/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 scale=0.001 0.001 0.001
- link mobile_wx250s/wrist_link: geometry collision mesh filename=package://clik1_node_pkg/model/meshes/mobile_wx250s_meshes/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 scale=0.001 0.001 0.001; visual mesh filename=package://clik1_node_pkg/model/meshes/mobile_wx250s_meshes/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 scale=0.001 0.001 0.001

Commit message: Updated mesh file path for gripper

File: model/wx250s.urdf (robot description, URDF)
Before this commit: robot mobile_wx250s, 14 links, 13 joints
Links:
- link mobile_wx250s/right_finger_link: geometry collision mesh filename=package://clik1_node_pkg/model/meshes/mobile_wx250s_meshes/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 scale=0.001 0.001 0.001; visual mesh filename=package://clik1_node_pkg/model/meshes/mobile_wx250s_meshes/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 scale=0.001 0.001 0.001
